File: ProgrammableLM317.kicad_pcb (KiCad board)
At the start: 2 copper layers, 49.5 x 49.5 mm, 28 parts, among them IC1 ATTINY85, K1 CONN_3, P1 CONN_2, P2 CONN_2, U1 LM317, U2 LM358, U3 MCP4801, U4 7805

Commit message: adding protection diodes to board layout
Parts:
- removed C10, C11: 0.1uF, CERCAP_2_059A
- added D1: 1N4001, DIODE_3_059A, F.Cu at (155.6, 146.1)
- added D2: 1N4001, DIODE_3_059A, F.Cu at (152.4, 154.9)
- IC1: value ATTINY85 -> ATTINY85-P
- moved C9 5.08 mm to (158.1, 158.1)
- moved C8 2.54 mm to (160.7, 158.1)
- moved C6 1.27 mm to (157.5, 135.3)
Routing:
- net Vout: track 28.8 -> 37.7 mm
- net 5V: track 92.3 -> 88.5 mm
- net Vcc: track 90.8 -> 92.6 mm
- net N-0000016: track 34.9 -> 36.4 mm
Other:
- board text added: "Programmable LM317 v2"
- board text added: "v2"
