File: ProgrammableLM317.sch (KiCad schematic (older format))
At the start: 25 parts, among them IC1 ATTINY85-P, K1 CONN_3, P1 CONN_2, P2 CONN_2, U1 LM317, U2 LM358, U3 MCP4801, U4 7805

Commit message: removing superfluous capacitors
Parts:
- removed C10, C11: 0.1uF, ~, symbol C_CER
- added D1, D2: 1N4001, ~, symbol DIODE
Connections:
- wire segments 82 -> 101
Other:
- note added: "Safely terminating the unused op amp..."
- moved on the sheet: C2, C3, C4, C6, C7, C8, C9, IC1, P2, R1, R2, R3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

Commit message: rearranging schematic.
Connections:
- wire segments 101 -> 86
Other:
- moved on the sheet: C1, C2, C3, C4, C6, C7, C8, C9, D1, D2, IC1, K1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
